File: design_files/AST1020.brd (EAGLE design)
At the start: 10 x 10 mm, 8 parts, among them J2 SM05B, J3 SH-7010TA, U1 SX1505I087TRT

Commit message: updated documentation
Parts:
- removed J3: SH-7010TA, tinycircuits:SH-7000
- added J1: SM05B, tinycircuits:JST_SH_5X1_EDGE
- C1: value 0.1uF -> 1uF
- J2: value SM05B -> SH-7010TA; device tinycircuits:JST_SH_5X1 -> tinycircuits:SH-7000
- moved J2 1.57 mm to (20.0, 13.7), flipped to the bottom
- renumbered R5 to R2, R7 to R1
Connections:
- net A: now also J2.8; no longer J3.8
- net B: now also J2.4; no longer J3.4
- net C: now also J2.2; no longer J3.2
- net D: now also J2.1; no longer J3.1
- net GND: now also J1.1, J2.C1, J2.C2; no longer J2.1, J3.C1, J3.C2
- net INT: now also J1.5; no longer J2.5
- net SCL: now also J1.3; no longer J2.3
- net SDA: now also J1.4; no longer J2.4
- net VCC: now also J1.2; no longer J2.2
Other:
- board text added: "Wireling Rotary Switch"
- board text removed: "Rotary Switch Board"
Changed lines of the file:
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@@
 <layer number="59" name="Invisible" color="7" fill="1" visible="no" active="no"/>
 <layer number="61" name="stand" color="7" fill="1" visible="no" active="no"/>
+<layer number="88" name="SimResults" color="9" fill="1" visible="yes" active="yes"/>
+<layer number="89" name="SimProbes" color="9" fill="1" visible="yes" active="yes"/>
 <layer number="90" name="Modules" color="5" fill="1" visible="yes" active="yes"/>
 <layer number="91" name="Nets" color="2" fill="1" visible="no" active="no"/>
@@
 <layer number="158" name="bResistor" color="7" fill="1" visible="yes" active="yes"/>
 <layer number="159" name="henwayCAP" color="13" fill="1" visible="yes" active="yes"/>
+<layer number="160" name="IDFDebug" color="7" fill="1" visible="yes" active="yes"/>
 <layer number="191" name="mNets" color="7" fill="1" visible="no" active="no"/>
 <layer number="192" name="mBusses" color="7" fill="1" visible="no" active="no"/>
@@
 <wire x1="0" y1="40.8" x2="0" y2="0" width="0.127" layer="48"/>
 <dimension x1="15" y1="20" x2="25" y2="20" x3="20" y3="21.454653125" layer="48"/>
-<text x="38.111025" y="4.365003125" size="0.889" layer="48">Rotary Switch Board</text>
+<text x="38.111025" y="4.365003125" size="0.889" layer="48">Wireling Rotary Switch</text>
 <text x="34.986825" y="1.7714" size="0.889" layer="48">AS-PCB-AST1020</text>
 <text x="57.3810375" y="1.6952" size="0.889" layer="48">3</text>
@@
 <attribute name="NO_BOM" value="TRUE" x="34" y="0" size="1.778" layer="27" display="off"/>
 </element>
-<element name="J3" library="tinycircuits" package="SH-7000" value="SH-7010TA" x="20" y="13.7" rot="MR0">
+<element name="J2" library="tinycircuits" package="SH-7000" value="SH-7010TA" x="20" y="13.7" rot="MR0">
 <attribute name="PARTNO" value="AS-ITM-00295" x="20" y="13.7" size="1.778" layer="28" rot="MR0" display="off"/>
 <attribute name="VALUE" value="SH-7010TA" x="20" y="13.7" size="1.778" layer="28" rot="MR0" display="off"/>
-</element>
-<element name="J2" library="tinycircuits" package="JST_SH_5X1" value="SM05B" x="20" y="12.125">
+<attribute name="PNPROTATION" value="0" x="20" y="13.7" size="1.778" layer="28" rot="MR0" display="off"/>
+</element>
+<element name="J1" library="tinycircuits" package="JST_SH_5X1_EDGE" value="SM05B" x="20" y="12.125">
 <attribute name="PARTNO" value="AS-ITM-00340" x="20" y="12.125" size="1.778" layer="27" display="off"/>
 <attribute name="VALUE" value="SM05B" x="20" y="12.125" size="1.778" layer="27" display="off"/>
@@
 <attribute name="VALUE" value="SX1505I087TRT" x="19.8" y="17.8" size="1.778" layer="27" display="off"/>
 </element>
-<element name="R5" library="tinycircuits" package="0402" value="10.0K" x="20" y="19" rot="MR0">
+<element name="R2" library="tinycircuits" package="0402" value="10.0K" x="20" y="19" rot="MR0">
 <attribute name="PARTNO" value="AS-ITM-00032" x="20" y="19" size="1.778" layer="28" rot="MR0" display="off"/>
 <attribute name="VALUE" value="10.0K" x="20" y="19" size="1.778" layer="28" rot="MR0" display="off"/>
 </element>
-<element name="R7" library="tinycircuits" package="0402" value="1.00K" x="22.9" y="15.9" rot="R180">
+<element name="R1" library="tinycircuits" package="0402" value="1.00K" x="22.9" y="15.9" rot="R180">
 <attribute name="PARTNO" value="AS-ITM-00003" x="22.9" y="15.9" size="1.778" layer="27" rot="R180" display="off"/>
 <attribute name="VALUE" value="1.00K" x="22.9" y="15.9" size="1.778" layer="27" rot="R180" display="off"/>
 </element>
-<element name="C1" library="tinycircuits" package="C0402" value="0.1uF" x="17.1" y="15.2" rot="R270">
-<attribute name="PARTNO" value="AS-ITM-00008" x="17.1" y="15.2" size="1.778" layer="27" rot="R270" display="off"/>
-<attribute name="VALUE" value="0.1uF" x="17.1" y="15.2" size="1.778" layer="27" rot="R270" display="off"/>
+<element name="C1" library="tinycircuits" package="C0402" value="1uF" x="17.1" y="15.2" rot="R270">
+<attribute name="PARTNO" value="AS-ITM-00105" x="17.1" y="15.2" size="1.778" layer="27" rot="R270" display="off"/>
+<attribute name="VALUE" value="1uF" x="17.1" y="15.2" size="1.778" layer="27" rot="R270" display="off"/>
 </element>
 <element name="C2" library="tinycircuits" package="C0402" value="0.1uF" x="23.8" y="17.1">
@@
 <vertex x="15" y="10"/>
 </polygon>
-<contactref element="J3" pad="C2"/>
-<contactref element="J3" pad="C1"/>
-<contactref element="J2" pad="1"/>
+<contactref element="J2" pad="C2"/>
+<contactref element="J2" pad="C1"/>
+<contactref element="J1" pad="1"/>
 <contactref element="U1" pad="PAD"/>
 <contactref element="U1" pad="8"/>
@@
 </signal>
 <signal name="SDA">
-<contactref element="J2" pad="4"/>
+<contactref element="J1" pad="4"/>
 <contactref element="U1" pad="2"/>
 <wire x1="18.35" y1="18.2" x2="17.7" y2="18.2" width="0.2032" layer="1"/>
@@
 </signal>
 <signal name="SCL">
-<contactref element="J2" pad="3"/>
+<contactref element="J1" pad="3"/>
 <contactref element="U1" pad="4"/>
 <wire x1="17.4" y1="17" x2="17.8" y2="17.4" width="0.2032" layer="1"/>
@@
 </signal>
 <signal name="VCC">
-<contactref element="J2" pad="2"/>
+<contactref element="J1" pad="2"/>
 <contactref element="U1" pad="17"/>
 <contactref element="U1" pad="7"/>
 <contactref element="U1" pad="14"/>
-<contactref element="R5" pad="1"/>
+<contactref element="R2" pad="1"/>
 <contactref element="U1" pad="16"/>
 <wire x1="20.2" y1="19.25" x2="20.2" y2="19.6" width="0.2032" layer="1"/>
@@
 </signal>
 <signal name="INT">
-<contactref element="J2" pad="5"/>
-<contactref element="R7" pad="1"/>
+<contactref element="J1" pad="5"/>
+<contactref element="R1" pad="1"/>
 <wire x1="22" y1="14.6" x2="22.8" y2="14.6" width="0.2032" layer="1"/>
 <wire x1="22.8" y1="14.6" x2="23.5" y2="15.3" width="0.2032" layer="1"/>
@@
 </signal>
 <signal name="C">
-<contactref element="J3" pad="2"/>
+<contactref element="J2" pad="2"/>
 <contactref element="U1" pad="15"/>
 <wire x1="21.25" y1="18.6" x2="21.7" y2="18.6" width="0.2032" layer="1"/>
@@
 <contactref element="U1" pad="10"/>
 <via x="21.3" y="15.8" extent="1-16" drill="0.381"/>
-<contactref element="J3" pad="8"/>
+<contactref element="J2" pad="8"/>
 <wire x1="23.25" y1="11.16" x2="21.54" y2="11.26" width="0.2032" layer="16"/>
 <wire x1="21.54" y1="11.26" x2="21.3" y2="11.5" width="0.2032" layer="16"/>
@@
 </signal>
 <signal name="B">
-<contactref element="J3" pad="4"/>
+<contactref element="J2" pad="4"/>
 <contactref element="U1" pad="6"/>
 <wire x1="19" y1="16.35" x2="18.45" y2="16.35" width="0.2032" layer="1"/>
@@
 <signal name="N$21">
 <contactref element="U1" pad="11"/>
-<contactref element="R7" pad="2"/>
+<contactref element="R1" pad="2"/>
 <wire x1="21.25" y1="17" x2="21.6" y2="17" width="0.2032" layer="1"/>
 <wire x1="21.6" y1="17" x2="22" y2="16.6" width="0.2032" layer="1"/>
@@
 <signal name="N$22">
 <contactref element="U1" pad="1"/>
-<contactref element="R5" pad="2"/>
+<contactref element="R2" pad="2"/>
 <wire x1="18.35" y1="18.6" x2="18" y2="18.6" width="0.2032" layer="1"/>
 <wire x1="18" y1="18.6" x2="17.8" y2="18.8" width="0.2032" layer="1"/>
@@
 </signal>
 <signal name="D">
-<contactref element="J3" pad="1"/>
+<contactref element="J2" pad="1"/>
 <wire x1="17.6" y1="16.6" x2="16.8" y2="16.6" width="0.2032" layer="1"/>
 <wire x1="16.8" y1="16.6" x2="16.3" y2="16.1" width="0.2032" layer="1"/>
