File: design_files/AST1020.sch (EAGLE design)
At the start: 7 parts, among them J2 SM05B, J3 SH-7010TA, U1 SX1505I087TRT

Commit message: updated documentation
Parts:
- removed J3: SH-7010TA, tinycircuits:AS-ITM-00295
- added J1: SM05B, tinycircuits:AS-ITM-00340EDGE
- C1: value 0.1uF -> 1uF; device tinycircuits:AS-ITM-00008 -> tinycircuits:AS-ITM-00105; PARTNO (none) -> AS-ITM-00105; VALUE (none) -> 1uF
- J2: value SM05B -> SH-7010TA; device tinycircuits:AS-ITM-00340 -> tinycircuits:AS-ITM-00295
- renumbered R5 to R2, R7 to R1
Connections:
- net A: now also J2.8; no longer J3.8
- net B: now also J2.4; no longer J3.4
- net C: now also J2.2; no longer J3.2
- net D: now also J2.1; no longer J3.1
- net GND: now also J1.1, J2.COM1, J2.COM2; no longer J2.1, J3.COM1, J3.COM2
- net INT: now also J1.5; no longer J2.5
- net SCL: now also J1.3; no longer J2.3
- net SDA: now also J1.4; no longer J2.4
- net VCC: now also J1.2; no longer J2.2
Other:
- note added: "Rotary Switch and I2C IO Expander"
- note added: "Variant: Standard - R"
- note added: "Wireling Rotary Switch"
- note removed: "Rotary Switch"
- note removed: "Rotary Switch Board"
- note removed: "Variant: Standard"
